Commit message: urdf changes

File: urdf/qut10_jackal_extras.urdf.xacro (robot description, xacro)
@@ -15,5 +15,12 @@
     <parent link="mid_mount" />
     <child link="sensors_link" />
-    <origin xyz="0 0 0"/>
+    <origin xyz="-0.015 0 0.005"/>
+  </joint>
+<!-- VLP16 Link -->
+   <link name="velodyne"/>
+  <joint name="velodyne_to_mount" type="fixed">
+    <parent link="mid_mount" />
+    <child link="velodyne" />
+    <origin xyz="0.0701 0.00134 0.114"/>
   </joint>
 </robot>

Commit message: urdf update

File: urdf/qut10_jackal_extras.urdf.xacro (robot description, xacro)
@@ -24,3 +24,17 @@
     <origin xyz="0.0701 0.00134 0.114"/>
   </joint>
+<!-- Front Laser -->
+   <link name="front_laser"/>
+  <joint name="velodyne_to_mount" type="fixed">
+    <parent link="front_mount" />
+    <child link="front_laser" />
+    <origin xyz="0 0 0"/>
+  </joint>
+<!-- Rear Laser -->
+   <link name="rear_laser"/>
+  <joint name="velodyne_to_mount" type="fixed">
+    <parent link="rear_mount" />
+    <child link="rear_laser" />
+    <origin xyz="0 0 0"/>
+  </joint>
 </robot>

Commit message: urdf update

File: urdf/qut10_jackal_extras.urdf.xacro (robot description, xacro)
@@ -26,5 +26,5 @@
 <!-- Front Laser -->
    <link name="front_laser"/>
-  <joint name="velodyne_to_mount" type="fixed">
+  <joint name="laser_to_fmount" type="fixed">
     <parent link="front_mount" />
     <child link="front_laser" />
@@ -33,5 +33,5 @@
 <!-- Rear Laser -->
    <link name="rear_laser"/>
-  <joint name="velodyne_to_mount" type="fixed">
+  <joint name="laser_to_rmount" type="fixed">
     <parent link="rear_mount" />
     <child link="rear_laser" />

Commit message: urdf update

File: urdf/qut10_jackal_extras.urdf.xacro (robot description, xacro)
@@ -36,5 +36,5 @@
     <parent link="rear_mount" />
     <child link="rear_laser" />
-    <origin xyz="0 0 0"/>
+    <origin xyz="0 0 0" rpy="0 0 3.14159"/>
   </joint>
 </robot>

Commit message: urdf changes

File: urdf/qut10_jackal_extras.urdf.xacro (robot description, xacro)
@@ -24,18 +24,17 @@
     <origin xyz="0.0701 0.00134 0.114"/>
   </joint>
-<!-- Front Laser
+<!-- Front Laser  -->
    <link name="front_laser"/>
   <joint name="laser_to_fmount" type="fixed">
-    <parent link="front_mount" />
+    <parent link="front_ust10_laser" />
     <child link="front_laser" />
     <origin xyz="0 0 0"/>
   </joint>
-<!- Rear Laser
+<!-- Rear Laser  -->
    <link name="rear_laser"/>
   <joint name="laser_to_rmount" type="fixed">
-    <parent link="rear_mount" />
+    <parent link="rear_ust10_laser" />
     <child link="rear_laser" />
-    <origin xyz="0 0 0" rpy="0 0 3.14159"/>
+    <origin xyz="0 0 0" rpy="0 0 0"/>
   </joint>
--->
 </robot>

Commit message: urdf changes

File: urdf/qut10_jackal_extras.urdf.xacro (robot description, xacro)
@@ -24,17 +24,3 @@
     <origin xyz="0.0701 0.00134 0.114"/>
   </joint>
-<!-- Front Laser  -->
-   <link name="front_laser"/>
-  <joint name="laser_to_fmount" type="fixed">
-    <parent link="front_ust10_laser" />
-    <child link="front_laser" />
-    <origin xyz="0 0 0"/>
-  </joint>
-<!-- Rear Laser  -->
-   <link name="rear_laser"/>
-  <joint name="laser_to_rmount" type="fixed">
-    <parent link="rear_ust10_laser" />
-    <child link="rear_laser" />
-    <origin xyz="0 0 0" rpy="0 0 0"/>
-  </joint>
 </robot>

Commit message: Add preliminary occam frame

File: urdf/qut10_jackal_extras.urdf.xacro (robot description, xacro)
@@ -24,3 +24,10 @@
     <origin xyz="0.0701 0.00134 0.114"/>
   </joint>
+<!-- Occam camera -->
+   <link name="occam"/>
+  <joint name="occam_to_mount" type="fixed">
+    <parent link="mid_mount" />
+    <child link="occam" />
+    <origin xyz="0.0701 0.00134 0.219"/>
+  </joint>
 </robot>

Commit message: Add transforms for front left/right cameras

File: urdf/qut10_jackal_extras.urdf.xacro (robot description, xacro)
@@ -31,3 +31,17 @@
     <origin xyz="0.0701 0.00134 0.219"/>
   </joint>
+<!-- Right front camera -->
+   <link name="right_cam"/>
+  <joint name="right_cam_to_mount" type="fixed">
+    <parent link="front_mount" />
+    <child link="right_cam" />
+    <origin xyz="0.1 -0.122 0.075"/>
+  </joint>
+<!-- Left front camera -->
+   <link name="left_cam"/>
+  <joint name="left_cam_to_mount" type="fixed">
+    <parent link="front_mount" />
+    <child link="left_cam" />
+    <origin xyz="0.1 0.122 0.075"/>
+  </joint>
 </robot>

Commit message: Changes on robot

File: urdf/qut10_jackal_extras.urdf.xacro (robot description, xacro)
@@ -3,5 +3,5 @@
 <robot
  xmlns:xacro="http://ros.org/wiki/xacro">
-<!-- Sensors -->
+  <!-- Sensors -->
   <link name="sensors_link">
    <visual>
@@ -17,6 +17,6 @@
     <origin xyz="-0.015 0 0.005"/>
   </joint>
-<!-- VLP16 Link -->
-   <link name="velodyne"/>
+  <!-- VLP16 Link -->
+  <link name="velodyne"/>
   <joint name="velodyne_to_mount" type="fixed">
     <parent link="mid_mount" />
@@ -24,6 +24,6 @@
     <origin xyz="0.0701 0.00134 0.114"/>
   </joint>
-<!-- Occam camera -->
-   <link name="occam"/>
+  <!-- Occam camera -->
+  <link name="occam"/>
   <joint name="occam_to_mount" type="fixed">
     <parent link="mid_mount" />
@@ -31,17 +31,31 @@
     <origin xyz="0.0701 0.00134 0.219"/>
   </joint>
-<!-- Right front camera -->
-   <link name="right_cam"/>
+  <!-- Right front camera -->
+  <link name="right_cam"/>
   <joint name="right_cam_to_mount" type="fixed">
     <parent link="front_mount" />
     <child link="right_cam" />
-    <origin xyz="0.1 -0.122 0.075"/>
+    <origin xyz="0.17 -0.05 0.0"/>
   </joint>
-<!-- Left front camera -->
-   <link name="left_cam"/>
+  <!-- Left front camera -->
+  <link name="left_cam"/>
   <joint name="left_cam_to_mount" type="fixed">
     <parent link="front_mount" />
     <child link="left_cam" />
-    <origin xyz="0.1 0.122 0.075"/>
+    <origin xyz="0.17 0.05 0.0"/>
+  </joint>
+  <!-- Toposens -->
+  <link name="toposens">
+    <visual>
+      <geometry>
+        <mesh filename="package://toposens_description/meshes/TS3.dae" scale="0.001 0.001 0.001"/>
+      </geometry>
+      <origin xyz="-0.011 0.01 0"/>
+    </visual>
+  </link>
+  <joint name="toposens_to_mount" type="fixed">
+    <parent link="front_mount" />
+    <child link="toposens" />
+    <origin xyz="0.25 0.0 -0.03" rpy="3.1414 0 0"/>
   </joint>
 </robot>
